File: microCortex.kicad_pcb (KiCad board)
At the start: 4 copper layers, 60.1 x 22.9 mm, 31 parts, among them J1 Feather, J2 20021121-00010C4LF, SW1 KMR231NG LFS, U1 ATSAMD21G18A-AUT, U2 BQ24075, U3 BQ27441DRZR-G1A, U4 TLV70033_WSON6, U5 BMP280, Y1 Crystal

Commit message: Added logo
Parts:
- added G***: LOGO, microCortexLogo:microCortexLogo, F.Cu at (191.9, 96.5)
- added G***: LOGO, microCortexLogo:microCortexLogo, F.Cu at (0.00, 0.00)

Commit message: Updated pcb
Parts:
- removed the G*** at (0.00, 0.00)
